Commit message: Spawn 4 bots (Sliding bug if more than 1 bot is spawned)

File: src/swarm_simulation/urdf/redbot.xacro (robot description, xacro)
@@ -7,5 +7,5 @@
     <link name="base_link">
     <!-- Altered Inertial values using trial and error process for stablilization of bot-->
-        <xacro:box_inertia m = "2.0" x = "0.14" y = "0.14" z = "0.2" />
+        <xacro:box_inertia m = "1.0" x = "0.14" y = "0.14" z = "0.2" />
         <!-- <inertial> -->
         <!--     <origin rpy="0 0 0" xyz="0 0 0" /> -->

File: src/swarm_simulation/urdf/rim.urdf.xacro (robot description, xacro)
@@ -8,5 +8,5 @@
 			<inertial>
 				<origin xyz="0 0 -0.000343"/>
-				<mass value="0.2253637"/> <!-- 0.00835758 -->
+				<mass value="0.00835758"/> <!-- 0.00835758 -->
 				<inertia
 				ixx="8.63684e-07"

File: src/swarm_simulation/urdf/roller.urdf.xacro (robot description, xacro)
@@ -6,5 +6,5 @@
 		<link name="roller_${name}_rim_${parent}_link">
 			<inertial>
-				<mass value="0.001107675"/>
+				<mass value="0.00113845"/>
 				<!-- 0.00113845 -->
 				<!-- 0.001707675 -->

Commit message: Added AruCo detector launch

File: src/swarm_simulation/urdf/redbot.xacro (robot description, xacro)
@@ -28,5 +28,5 @@
     <link name = "aruco_tag">
         <visual>
-            <origin rpy = "0 0 0" xyz = "0 0 0.1" />
+            <origin rpy = "0 0 1.57" xyz = "0 0 0.1" />
             <geometry>
                 <mesh filename="package://swarm_simulation/models/aruco_tags/ID_1.dae" scale='1 1 1' />
