Commit message: Added Teleop script for swarm robots

File: src/swarm_simulation/urdf/bluebot.xacro (robot description, xacro)
@@ -47,5 +47,5 @@
     <!-- Left wheel link -->
     <xacro:rim_macro
-    name="left"
+    name="right"
     color="0 1 0"
     xyz="0.0585 0 -.0735"
@@ -53,5 +53,5 @@
     <!-- Right Wheel link  -->
     <xacro:rim_macro
-    name="right"
+    name="left"
     color="0 1 0"
     xyz="-0.0590 0 -.0735"

File: src/swarm_simulation/urdf/greenbot.xacro (robot description, xacro)
@@ -47,5 +47,5 @@
     <!-- Left wheel link -->
     <xacro:rim_macro
-    name="left"
+    name="right"
     color="0 1 0"
     xyz="0.0585 0 -.0735"
@@ -53,5 +53,5 @@
     <!-- Right Wheel link  -->
     <xacro:rim_macro
-    name="right"
+    name="left"
     color="0 1 0"
     xyz="-0.0590 0 -.0735"

File: src/swarm_simulation/urdf/greybot.xacro (robot description, xacro)
@@ -47,5 +47,5 @@
     <!-- Left wheel link -->
     <xacro:rim_macro
-    name="left"
+    name="right"
     color="0 1 0"
     xyz="0.0585 0 -.0735"
@@ -53,5 +53,5 @@
     <!-- Right Wheel link  -->
     <xacro:rim_macro
-    name="right"
+    name="left"
     color="0 1 0"
     xyz="-0.0590 0 -.0735"

File: src/swarm_simulation/urdf/redbot.xacro (robot description, xacro)
@@ -10,5 +10,5 @@
         <inertial>
             <origin rpy="0 0 0" xyz="0 0 0" />
-            <mass value="0.9" />
+            <mass value="0.9" /> <!-- 0.9 -->
             <inertia ixx="0.000070003" ixy="0.0" ixz="0.0" iyy="0.000070003" iyz="0.0" izz="0.000040" />
             <!-- <inertia ixx="0" ixy="-0.0" ixz="-1e-06" iyy="0" iyz="0" izz="0" /> -->
@@ -47,5 +47,5 @@
     <!-- Left wheel link -->
     <xacro:rim_macro
-    name="left"
+    name="right"
     color="0 1 0"
     xyz="0.0585 0 -.0735"
@@ -53,5 +53,5 @@
     <!-- Right Wheel link  -->
     <xacro:rim_macro
-    name="right"
+    name="left"
     color="0 1 0"
     xyz="-0.0590 0 -.0735"
@@ -60,5 +60,5 @@
     <gazebo>
 		<plugin name="gazebo_ros_control" filename="libgazebo_ros_control.so">
-		<robotNamespace>redbot</robotNamespace>
+		<robotNamespace>/redbot</robotNamespace>
 		</plugin>
 	</gazebo>

File: src/swarm_simulation/urdf/rim.urdf.xacro (robot description, xacro)
@@ -94,5 +94,5 @@
 			<actuator name="rim_${name}_motor">
 				<hardwareInterface>hardware_interface/VelocityJointInterface</hardwareInterface>
-				<mechanicalReduction>1</mechanicalReduction>
+				<mechanicalReduction>100</mechanicalReduction>
 			</actuator>
 		</transmission>

Commit message: Added Aruco Tags on Robots

File: src/swarm_simulation/urdf/bluebot.xacro (robot description, xacro)
@@ -27,4 +27,12 @@
         </collision>
     </link>
+    <link name = "aruco_tag">
+        <visual>
+            <origin rpy = "0 0 0" xyz = "0 0 0.1" />
+            <geometry>
+                <mesh filename="package://swarm_simulation/models/aruco_tags/ID_3.dae" scale='1 1 1' />
+            </geometry>
+        </visual>
+    </link>
     <!-- Dummy link -->
     <joint name="dummy_joint" type="fixed">
@@ -33,7 +41,13 @@
         <origin xyz = "0 0 0"/>
     </joint>
+    <joint name="aruco_joint" type="fixed">
+        <parent link ="base_link" />
+        <child link = "aruco_tag" />
+        <origin rpy = "0 0 0" xyz = "0 0 0" />
+    </joint>
     <!-- Front wheel link -->
     <xacro:rim_macro
     name="front"
+    robot_name = "bluebot"
     color="0 1 0"
     xyz="0 0.0585 -.0735"
@@ -42,4 +56,5 @@
     <xacro:rim_macro
     name="rear"
+    robot_name = "bluebot"
     color="0 1 0"
     xyz="0 -0.0595 -.0735"
@@ -48,4 +63,5 @@
     <xacro:rim_macro
     name="right"
+    robot_name = "bluebot"
     color="0 1 0"
     xyz="0.0585 0 -.0735"
@@ -54,4 +70,5 @@
     <xacro:rim_macro
     name="left"
+    robot_name = "bluebot"
     color="0 1 0"
     xyz="-0.0590 0 -.0735"

File: src/swarm_simulation/urdf/greenbot.xacro (robot description, xacro)
@@ -27,4 +27,12 @@
         </collision>
     </link>
+    <link name = "aruco_tag">
+        <visual>
+            <origin rpy = "0 0 0" xyz = "0 0 0.1" />
+            <geometry>
+                <mesh filename="package://swarm_simulation/models/aruco_tags/ID_2.dae" scale='1 1 1' />
+            </geometry>
+        </visual>
+    </link>
     <!-- Dummy link -->
     <joint name="dummy_joint" type="fixed">
@@ -33,7 +41,13 @@
         <origin xyz = "0 0 0"/>
     </joint>
+    <joint name="aruco_joint" type="fixed">
+        <parent link ="base_link" />
+        <child link = "aruco_tag" />
+        <origin rpy = "0 0 0" xyz = "0 0 0" />
+    </joint>
     <!-- Front wheel link -->
     <xacro:rim_macro
     name="front"
+    robot_name = "greenbot"
     color="0 1 0"
     xyz="0 0.0585 -.0735"
@@ -42,4 +56,5 @@
     <xacro:rim_macro
     name="rear"
+    robot_name = "greenbot"
     color="0 1 0"
     xyz="0 -0.0595 -.0735"
@@ -48,4 +63,5 @@
     <xacro:rim_macro
     name="right"
+    robot_name = "greenbot"
     color="0 1 0"
     xyz="0.0585 0 -.0735"
@@ -54,4 +70,5 @@
     <xacro:rim_macro
     name="left"
+    robot_name = "greenbot"
     color="0 1 0"
     xyz="-0.0590 0 -.0735"

File: src/swarm_simulation/urdf/greybot.xacro (robot description, xacro)
@@ -27,4 +27,12 @@
         </collision>
     </link>
+    <link name = "aruco_tag">
+        <visual>
+            <origin rpy = "0 0 0" xyz = "0 0 0.1" />
+            <geometry>
+                <mesh filename="package://swarm_simulation/models/aruco_tags/ID_4.dae" scale='1 1 1' />
+            </geometry>
+        </visual>
+    </link>
     <!-- Dummy link -->
     <joint name="dummy_joint" type="fixed">
@@ -33,7 +41,13 @@
         <origin xyz = "0 0 0"/>
     </joint>
+    <joint name="aruco_joint" type="fixed">
+        <parent link ="base_link" />
+        <child link = "aruco_tag" />
+        <origin rpy = "0 0 0" xyz = "0 0 0" />
+    </joint>
     <!-- Front wheel link -->
     <xacro:rim_macro
     name="front"
+    robot_name = "greybot"
     color="0 1 0"
     xyz="0 0.0585 -.0735"
@@ -42,4 +56,5 @@
     <xacro:rim_macro
     name="rear"
+    robot_name = "greybot"
     color="0 1 0"
     xyz="0 -0.0595 -.0735"
@@ -48,4 +63,5 @@
     <xacro:rim_macro
     name="right"
+    robot_name = "greybot"
     color="0 1 0"
     xyz="0.0585 0 -.0735"
@@ -54,4 +70,5 @@
     <xacro:rim_macro
     name="left"
+    robot_name = "greybot"
     color="0 1 0"
     xyz="-0.0590 0 -.0735"

File: src/swarm_simulation/urdf/redbot.xacro (robot description, xacro)
@@ -27,4 +27,12 @@
         </collision>
     </link>
+    <link name = "aruco_tag">
+        <visual>
+            <origin rpy = "0 0 0" xyz = "0 0 0.1" />
+            <geometry>
+                <mesh filename="package://swarm_simulation/models/aruco_tags/ID_1.dae" scale='1 1 1' />
+            </geometry>
+        </visual>
+    </link>
     <!-- Dummy link -->
     <joint name="dummy_joint" type="fixed">
@@ -33,7 +41,13 @@
         <origin xyz = "0 0 0"/>
     </joint>
+    <joint name="aruco_joint" type="fixed">
+        <parent link ="base_link" />
+        <child link = "aruco_tag" />
+        <origin rpy = "0 0 0" xyz = "0 0 0" />
+    </joint>
     <!-- Front wheel link -->
     <xacro:rim_macro
     name="front"
+    robot_name = "redbot"
     color="0 1 0"
     xyz="0 0.0585 -.0735"
@@ -42,4 +56,5 @@
     <xacro:rim_macro
     name="rear"
+    robot_name = "redbot"
     color="0 1 0"
     xyz="0 -0.0595 -.0735"
@@ -48,4 +63,5 @@
     <xacro:rim_macro
     name="right"
+    robot_name = "redbot"
     color="0 1 0"
     xyz="0.0585 0 -.0735"
@@ -54,4 +70,5 @@
     <xacro:rim_macro
     name="left"
+    robot_name = "redbot"
     color="0 1 0"
     xyz="-0.0590 0 -.0735"

File: src/swarm_simulation/urdf/rim.urdf.xacro (robot description, xacro)
@@ -4,6 +4,6 @@
 <xacro:macro
 	name="rim_macro"
-	params="name color xyz rpy">
-		<link name="rim_${name}_link">
+	params="name robot_name color xyz rpy">
+		<link name="${robot_name}_rim_${name}_link">
 			<inertial>
 				<origin xyz="0 0 -0.000343"/>
@@ -21,5 +21,5 @@
 					<mesh filename="package://swarm_simulation/models/wheel/meshes/rim.stl" scale = "1.5 1.5 1.5"/>
 				</geometry>
-				<material name="rim_${name}_material">
+				<material name="${robot_name}_rim_${name}_material">
 					<color rgba="${color} 1"/>
 				</material>
@@ -32,8 +32,8 @@
 		</link>
 		<joint
-			name="rim_${name}_joint"
+			name="${robot_name}_rim_${name}_joint"
 			type="continuous">
 			<parent link="base_link" />
-			<child link="rim_${name}_link" />
+			<child link="${robot_name}_rim_${name}_link" />
 			<axis xyz="0 0 1"/>
 			<origin xyz="${xyz}" rpy="${rpy}"/>
@@ -41,4 +41,5 @@
 		<xacro:roller_macro
 			parent="${name}"
+			robot_name = "${robot_name}"
 			name="e"
 			xyz="0.02035 0 0.0085"
@@ -47,4 +48,5 @@
 		<xacro:roller_macro
 			parent="${name}"
+			robot_name = "${robot_name}"
 			name="ne"
 			xyz="0.01429 0.01429 -0.0085"
@@ -53,4 +55,5 @@
 		<xacro:roller_macro
 			parent="${name}"
+			robot_name = "${robot_name}"
 			name="n"
 			xyz="0 0.02035 0.0085"
@@ -59,4 +62,5 @@
 		<xacro:roller_macro
 			parent="${name}"
+			robot_name = "${robot_name}"
 			name="nw"
 			xyz="-0.01429 0.01429 -0.0085"
@@ -65,4 +69,5 @@
 		<xacro:roller_macro
 			parent="${name}"
+			robot_name = "${robot_name}"
 			name="w"
 			xyz="-0.02035 0 0.0085"
@@ -71,4 +76,5 @@
 		<xacro:roller_macro
 			parent="${name}"
+			robot_name = "${robot_name}"
 			name="sw"
 			xyz="-0.01429 -0.01429 -0.0085"
@@ -77,4 +83,5 @@
 		<xacro:roller_macro
 			parent="${name}"
+			robot_name = "${robot_name}"
 			name="s"
 			xyz="0 -0.02035 0.0085"
@@ -83,32 +90,19 @@
 		<xacro:roller_macro
 			parent="${name}"
+			robot_name = "${robot_name}"
 			name="se"
 			xyz="0.01429 -0.01429 -0.0085"
 			rpy="-1.570796326794896 0 -0.7853981633974483"
 		/>
-		<transmission name="rim_${name}_transmission">
+		<transmission name="${robot_name}_rim_${name}_transmission">
 			<type>transmission_interface/SimpleTransmission</type>
-			<joint name="rim_${name}_joint">
+			<joint name="${robot_name}_rim_${name}_joint">
 				<hardwareInterface>hardware_interface/VelocityJointInterface</hardwareInterface>
 			</joint>
-			<actuator name="rim_${name}_motor">
+			<actuator name="${robot_name}_rim_${name}_motor">
 				<hardwareInterface>hardware_interface/VelocityJointInterface</hardwareInterface>
-				<mechanicalReduction>100</mechanicalReduction>
+				<mechanicalReduction>1</mechanicalReduction>
 			</actuator>
 		</transmission>
 	</xacro:macro>
 </robot>
-<!-- xyz="0.01529 -0.01529 -0.0085" -->
-<!-- ixx="6.63684e-07"
-ixy="0"
-ixz="0"
-iyy="6.63684e-07"
-iyz="0"
-izz="9.40333e-07" -->
-<!-- Scale : 1.5 -->
-<!-- ixx="9.95526e-07"
-ixy="0"
-ixz="0"
-iyy="9.95526e-07"
-iyz="0"
-izz="14.104995e-07" -->

File: src/swarm_simulation/urdf/roller.urdf.xacro (robot description, xacro)
@@ -3,10 +3,11 @@
 <xacro:macro
 	name="roller_macro"
-	params="parent name xyz rpy">
+	params="parent robot_name name xyz rpy">
 		<link name="roller_${name}_rim_${parent}_link">
 			<inertial>
-				<mass value="0.001107675"/>
+				<mass value="0.002007675"/>
 				<!-- 0.00113845 -->
 				<!-- 0.001707675 -->
+				<!-- 0.001107675 -->
 				<inertia
 				ixx="10.53776e-08"
@@ -35,5 +36,5 @@
   	</gazebo>
 		<joint name="roller_${name}_rim_${parent}_joint" type="continuous">
-			<parent link="rim_${parent}_link"/>
+			<parent link="${robot_name}_rim_${parent}_link"/>
 			<child link="roller_${name}_rim_${parent}_link"/>
 			<axis xyz="0 0 1"/>
