Commit message: Fixed Roller independent spinning by implementing PID control

File: src/swarm_simulation/urdf/bluebot.xacro (robot description, xacro)
@@ -6,12 +6,6 @@
     <link name="dummy"> </link>
     <link name="base_link">
-    <!-- Altered Inertial values using trial and error process for stablilization of bot-->
-        <!-- <xacro:box_inertia m = "0.80" x = "0.085" y = "-0.10" z = "0.05" /> -->
-        <inertial>
-            <origin rpy="0 0 0" xyz="0 0 0" />
-            <mass value="0.9" />
-            <inertia ixx="0.000070003" ixy="0.0" ixz="0.0" iyy="0.000070003" iyz="0.0" izz="0.000040" />
-            <!-- <inertia ixx="0" ixy="-0.0" ixz="-1e-06" iyy="0" iyz="0" izz="0" /> -->
-        </inertial>
+        <!-- Intertial Values Using MACRO (Mass Adjusted As Required)  -->
+        <xacro:box_inertia m="2.0" x="0.14" y="0.14" z="0.2" />
         <visual>
             <origin rpy="0 0 0" xyz="0 0 0" />
@@ -27,7 +21,7 @@
         </collision>
     </link>
-    <link name = "aruco_tag">
+    <link name="aruco_tag">
         <visual>
-            <origin rpy = "0 0 0" xyz = "0 0 0.1" />
+            <origin rpy="0 0 0" xyz="0 0 0.1" />
             <geometry>
                 <mesh filename="package://swarm_simulation/models/aruco_tags/ID_3.dae" scale='1 1 1' />
@@ -37,46 +31,46 @@
     <!-- Dummy link -->
     <joint name="dummy_joint" type="fixed">
-        <parent link="dummy"/>
-        <child link="base_link"/>
-        <origin xyz = "0 0 0"/>
+        <parent link="dummy" />
+        <child link="base_link" />
+        <origin xyz="0 0 0" />
     </joint>
     <joint name="aruco_joint" type="fixed">
-        <parent link ="base_link" />
-        <child link = "aruco_tag" />
-        <origin rpy = "0 0 0" xyz = "0 0 0" />
+        <parent link="base_link" />
+        <child link="aruco_tag" />
+        <origin rpy="0 0 0" xyz="0 0 0" />
     </joint>
     <!-- Front wheel link -->
     <xacro:rim_macro
-    name="front"
-    robot_name = "bluebot"
-    color="0 1 0"
-    xyz="0 0.0585 -.0735"
-    rpy="1.570796326794896 0.05 0"/>
+        name="front"
+        robot_name="bluebot"
+        color="0 1 0"
+        xyz="0 0.0585 -.0735"
+        rpy="1.570796326794896 0.05 0" />
     <!-- Rear wheel link -->
     <xacro:rim_macro
-    name="rear"
-    robot_name = "bluebot"
-    color="0 1 0"
-    xyz="0 -0.0595 -.0735"
-    rpy="1.570796326794896 0.05 3.14"/>
+        name="rear"
+        robot_name="bluebot"
+        color="0 1 0"
+        xyz="0 -0.0595 -.0735"
+        rpy="1.570796326794896 0.05 3.14" />
     <!-- Left wheel link -->
     <xacro:rim_macro
-    name="right"
-    robot_name = "bluebot"
-    color="0 1 0"
-    xyz="0.0585 0 -.0735"
-    rpy="1.570796326794896 0.05 -1.57"/>
+        name="right"
+        robot_name="bluebot"
+        color="0 1 0"
+        xyz="0.0585 0 -.0735"
+        rpy="1.570796326794896 0.05 -1.57" />
     <!-- Right Wheel link  -->
     <xacro:rim_macro
-    name="left"
-    robot_name = "bluebot"
-    color="0 1 0"
-    xyz="-0.0590 0 -.0735"
-    rpy="1.570796326794896 0.05 1.57"/>
+        name="left"
+        robot_name="bluebot"
+        color="0 1 0"
+        xyz="-0.0590 0 -.0735"
+        rpy="1.570796326794896 0.05 1.57" />
     <!-- Should install sudo apt-get install ros-noetic-ros-control ros-noetic-ros-controllers -->
     <gazebo>
-		<plugin name="gazebo_ros_control" filename="libgazebo_ros_control.so">
-		<robotNamespace>/bluebot</robotNamespace>
-		</plugin>
-	</gazebo>
+        <plugin name="gazebo_ros_control" filename="libgazebo_ros_control.so">
+            <robotNamespace>/bluebot</robotNamespace>
+        </plugin>
+    </gazebo>
 </robot>

File: src/swarm_simulation/urdf/greenbot.xacro (robot description, xacro)
@@ -6,12 +6,6 @@
     <link name="dummy"> </link>
     <link name="base_link">
-    <!-- Altered Inertial values using trial and error process for stablilization of bot-->
-        <!-- <xacro:box_inertia m = "0.80" x = "0.085" y = "-0.10" z = "0.05" /> -->
-        <inertial>
-            <origin rpy="0 0 0" xyz="0 0 0" />
-            <mass value="0.9" />
-            <inertia ixx="0.000070003" ixy="0.0" ixz="0.0" iyy="0.000070003" iyz="0.0" izz="0.000040" />
-            <!-- <inertia ixx="0" ixy="-0.0" ixz="-1e-06" iyy="0" iyz="0" izz="0" /> -->
-        </inertial>
+        <!-- Intertial Values Using MACRO (Mass Adjusted As Required)  -->
+        <xacro:box_inertia m="2.0" x="0.14" y="0.14" z="0.2" />
         <visual>
             <origin rpy="0 0 0" xyz="0 0 0" />
@@ -27,7 +21,7 @@
         </collision>
     </link>
-    <link name = "aruco_tag">
+    <link name="aruco_tag">
         <visual>
-            <origin rpy = "0 0 0" xyz = "0 0 0.1" />
+            <origin rpy="0 0 0" xyz="0 0 0.1" />
             <geometry>
                 <mesh filename="package://swarm_simulation/models/aruco_tags/ID_2.dae" scale='1 1 1' />
@@ -37,46 +31,46 @@
     <!-- Dummy link -->
     <joint name="dummy_joint" type="fixed">
-        <parent link="dummy"/>
-        <child link="base_link"/>
-        <origin xyz = "0 0 0"/>
+        <parent link="dummy" />
+        <child link="base_link" />
+        <origin xyz="0 0 0" />
     </joint>
     <joint name="aruco_joint" type="fixed">
-        <parent link ="base_link" />
-        <child link = "aruco_tag" />
-        <origin rpy = "0 0 0" xyz = "0 0 0" />
+        <parent link="base_link" />
+        <child link="aruco_tag" />
+        <origin rpy="0 0 0" xyz="0 0 0" />
     </joint>
     <!-- Front wheel link -->
     <xacro:rim_macro
-    name="front"
-    robot_name = "greenbot"
-    color="0 1 0"
-    xyz="0 0.0585 -.0735"
-    rpy="1.570796326794896 0.05 0"/>
+        name="front"
+        robot_name="greenbot"
+        color="0 1 0"
+        xyz="0 0.0585 -.0735"
+        rpy="1.570796326794896 0.05 0" />
     <!-- Rear wheel link -->
     <xacro:rim_macro
-    name="rear"
-    robot_name = "greenbot"
-    color="0 1 0"
-    xyz="0 -0.0595 -.0735"
-    rpy="1.570796326794896 0.05 3.14"/>
+        name="rear"
+        robot_name="greenbot"
+        color="0 1 0"
+        xyz="0 -0.0595 -.0735"
+        rpy="1.570796326794896 0.05 3.14" />
     <!-- Left wheel link -->
     <xacro:rim_macro
-    name="right"
-    robot_name = "greenbot"
-    color="0 1 0"
-    xyz="0.0585 0 -.0735"
-    rpy="1.570796326794896 0.05 -1.57"/>
+        name="right"
+        robot_name="greenbot"
+        color="0 1 0"
+        xyz="0.0585 0 -.0735"
+        rpy="1.570796326794896 0.05 -1.57" />
     <!-- Right Wheel link  -->
     <xacro:rim_macro
-    name="left"
-    robot_name = "greenbot"
-    color="0 1 0"
-    xyz="-0.0590 0 -.0735"
-    rpy="1.570796326794896 0.05 1.57"/>
+        name="left"
+        robot_name="greenbot"
+        color="0 1 0"
+        xyz="-0.0590 0 -.0735"
+        rpy="1.570796326794896 0.05 1.57" />
     <!-- Should install sudo apt-get install ros-noetic-ros-control ros-noetic-ros-controllers -->
     <gazebo>
-		<plugin name="gazebo_ros_control" filename="libgazebo_ros_control.so">
-		<robotNamespace>/greenbot</robotNamespace>
-		</plugin>
-	</gazebo>
+        <plugin name="gazebo_ros_control" filename="libgazebo_ros_control.so">
+            <robotNamespace>/greenbot</robotNamespace>
+        </plugin>
+    </gazebo>
 </robot>

File: src/swarm_simulation/urdf/greybot.xacro (robot description, xacro)
@@ -6,16 +6,11 @@
     <link name="dummy"> </link>
     <link name="base_link">
-    <!-- Altered Inertial values using trial and error process for stablilization of bot-->
-        <!-- <xacro:box_inertia m = "0.80" x = "0.085" y = "-0.10" z = "0.05" /> -->
-        <inertial>
-            <origin rpy="0 0 0" xyz="0 0 0" />
-            <mass value="0.9" />
-            <inertia ixx="0.000070003" ixy="0.0" ixz="0.0" iyy="0.000070003" iyz="0.0" izz="0.000040" />
-            <!-- <inertia ixx="0" ixy="-0.0" ixz="-1e-06" iyy="0" iyz="0" izz="0" /> -->
-        </inertial>
+        <!-- Intertial Values Using MACRO (Mass Adjusted As Required)  -->
+        <xacro:box_inertia m="2.0" x="0.14" y="0.14" z="0.2" />
         <visual>
             <origin rpy="0 0 0" xyz="0 0 0" />
             <geometry>
-                <mesh filename="package://swarm_simulation/models/Grey_bot/grey_bot.dae" scale="1 1 1" />
+                <mesh filename="package://swarm_simulation/models/Grey_bot/grey_bot.dae"
+                    scale="1 1 1" />
             </geometry>
         </visual>
@@ -23,11 +18,12 @@
             <origin rpy="0 0 0" xyz="0 0 0" />
             <geometry>
-                <mesh filename="package://swarm_simulation/models/Grey_bot/grey_bot.dae" scale="1 1 1" />
+                <mesh filename="package://swarm_simulation/models/Grey_bot/grey_bot.dae"
+                    scale="1 1 1" />
             </geometry>
         </collision>
     </link>
-    <link name = "aruco_tag">
+    <link name="aruco_tag">
         <visual>
-            <origin rpy = "0 0 0" xyz = "0 0 0.1" />
+            <origin rpy="0 0 0" xyz="0 0 0.1" />
             <geometry>
                 <mesh filename="package://swarm_simulation/models/aruco_tags/ID_4.dae" scale='1 1 1' />
@@ -37,46 +33,46 @@
     <!-- Dummy link -->
     <joint name="dummy_joint" type="fixed">
-        <parent link="dummy"/>
-        <child link="base_link"/>
-        <origin xyz = "0 0 0"/>
+        <parent link="dummy" />
+        <child link="base_link" />
+        <origin xyz="0 0 0" />
     </joint>
     <joint name="aruco_joint" type="fixed">
-        <parent link ="base_link" />
-        <child link = "aruco_tag" />
-        <origin rpy = "0 0 0" xyz = "0 0 0" />
+        <parent link="base_link" />
+        <child link="aruco_tag" />
+        <origin rpy="0 0 0" xyz="0 0 0" />
     </joint>
     <!-- Front wheel link -->
     <xacro:rim_macro
-    name="front"
-    robot_name = "greybot"
-    color="0 1 0"
-    xyz="0 0.0585 -.0735"
-    rpy="1.570796326794896 0.05 0"/>
+        name="front"
+        robot_name="greybot"
+        color="0 1 0"
+        xyz="0 0.0585 -.0735"
+        rpy="1.570796326794896 0.05 0" />
     <!-- Rear wheel link -->
     <xacro:rim_macro
-    name="rear"
-    robot_name = "greybot"
-    color="0 1 0"
-    xyz="0 -0.0595 -.0735"
-    rpy="1.570796326794896 0.05 3.14"/>
+        name="rear"
+        robot_name="greybot"
+        color="0 1 0"
+        xyz="0 -0.0595 -.0735"
+        rpy="1.570796326794896 0.05 3.14" />
     <!-- Left wheel link -->
     <xacro:rim_macro
-    name="right"
-    robot_name = "greybot"
-    color="0 1 0"
-    xyz="0.0585 0 -.0735"
-    rpy="1.570796326794896 0.05 -1.57"/>
+        name="right"
+        robot_name="greybot"
+        color="0 1 0"
+        xyz="0.0585 0 -.0735"
+        rpy="1.570796326794896 0.05 -1.57" />
     <!-- Right Wheel link  -->
     <xacro:rim_macro
-    name="left"
-    robot_name = "greybot"
-    color="0 1 0"
-    xyz="-0.0590 0 -.0735"
-    rpy="1.570796326794896 0.05 1.57"/>
+        name="left"
+        robot_name="greybot"
+        color="0 1 0"
+        xyz="-0.0590 0 -.0735"
+        rpy="1.570796326794896 0.05 1.57" />
     <!-- Should install sudo apt-get install ros-noetic-ros-control ros-noetic-ros-controllers -->
     <gazebo>
-		<plugin name="gazebo_ros_control" filename="libgazebo_ros_control.so">
-		<robotNamespace>/greybot</robotNamespace>
-		</plugin>
-	</gazebo>
+        <plugin name="gazebo_ros_control" filename="libgazebo_ros_control.so">
+            <robotNamespace>/greybot</robotNamespace>
+        </plugin>
+    </gazebo>
 </robot>

File: src/swarm_simulation/urdf/redbot.xacro (robot description, xacro)
@@ -7,11 +7,10 @@
     <link name="base_link">
     <!-- Altered Inertial values using trial and error process for stablilization of bot-->
-        <!-- <xacro:box_inertia m = "0.80" x = "0.085" y = "-0.10" z = "0.05" /> -->
-        <inertial>
-            <origin rpy="0 0 0" xyz="0 0 0" />
-            <mass value="0.9" /> <!-- 0.9 -->
-            <inertia ixx="0.000070003" ixy="0.0" ixz="0.0" iyy="0.000070003" iyz="0.0" izz="0.000040" />
-            <!-- <inertia ixx="0" ixy="-0.0" ixz="-1e-06" iyy="0" iyz="0" izz="0" /> -->
-        </inertial>
+        <xacro:box_inertia m = "2.0" x = "0.14" y = "0.14" z = "0.2" />
+        <!-- <inertial> -->
+        <!--     <origin rpy="0 0 0" xyz="0 0 0" /> -->
+        <!--     <mass value="0.9" /> <!-\- 0.9 -\-> -->
+        <!--     <inertia ixx="0.000070003" ixy="0.0" ixz="0.0" iyy="0.000070003" iyz="0.0" izz="0.000040" /> -->
+        <!--     <!-\- <inertia ixx="0" ixy="-0.0" ixz="-1e-06" iyy="0" iyz="0" izz="0" /> -\-> -->
         <visual>
             <origin rpy="0 0 0" xyz="0 0 0" />

File: src/swarm_simulation/urdf/rim.urdf.xacro (robot description, xacro)
@@ -8,5 +8,5 @@
 			<inertial>
 				<origin xyz="0 0 -0.000343"/>
-				<mass value="0.01253637"/> <!-- 0.00835758 -->
+				<mass value="0.2253637"/> <!-- 0.00835758 -->
 				<inertia
 				ixx="8.63684e-07"

File: src/swarm_simulation/urdf/roller.urdf.xacro (robot description, xacro)
@@ -6,5 +6,5 @@
 		<link name="roller_${name}_rim_${parent}_link">
 			<inertial>
-				<mass value="0.002007675"/>
+				<mass value="0.001107675"/>
 				<!-- 0.00113845 -->
 				<!-- 0.001707675 -->
